Commit message: zivid rviz

File: yumi_description/urdf/yumi.urdf (robot description, URDF)
Before this commit: robot yumi, 22 links, 21 joints
Links:
- added link zivid_optical_frame
Joints:
- added joint zivid_optical_joint: type fixed, parent yumi_base_link, child zivid_optical_frame, origin xyz=0.300 0 0.800 rpy=3.14 0 -1.5707

Commit message: point cloud in rviz

File: yumi_description/urdf/yumi.urdf (robot description, URDF)
Before this commit: robot yumi, 23 links, 22 joints
Joints:
- joint zivid_optical_joint: origin xyz=0.300 0 0.800 rpy=3.14 0 -1.5707 -> xyz=0.320 0 0.700 rpy=3.14 0 -1.5707

Commit message: added links for grip centers

File: yumi_description/urdf/yumi.urdf (robot description, URDF)
Before this commit: robot yumi, 23 links, 22 joints
Links:
- added link gripper_l_center
- added link gripper_r_center
Joints:
- added joint gripper_l_center_joint: type fixed, parent gripper_l_base, child gripper_l_center, origin xyz=0.0 0.0 0.1137 rpy=0 0 3.14159265359
- added joint gripper_r_center_joint: type fixed, parent gripper_r_base, child gripper_r_center, origin xyz=0.0 0.0 0.1137 rpy=0 0 3.14159265359
- joint zivid_optical_joint: origin xyz=0.320 0 0.700 rpy=3.14 0 -1.5707 -> xyz=0.300 0 0.800 rpy=3.14159 0.0 -1.57079

Commit message: correct base-camera calibration

File: yumi_description/urdf/yumi.urdf (robot description, URDF)
Before this commit: robot yumi, 25 links, 24 joints
Joints:
- joint zivid_optical_joint: origin xyz=0.300 0 0.800 rpy=3.14159 0.0 -1.57079 -> xyz=0.18817 0.06293 0.68891 rpy=-2.8595 -0.14513 -1.6163251

Commit message: adjusted grip center position

File: yumi_description/urdf/yumi.urdf (robot description, URDF)
Before this commit: robot yumi, 25 links, 24 joints
Joints:
- joint gripper_l_center_joint: origin xyz=0.0 0.0 0.1137 rpy=0 0 3.14159265359 -> xyz=0.0 0.0 0.13 rpy=0 0 3.14159265359
- joint gripper_r_center_joint: origin xyz=0.0 0.0 0.1137 rpy=0 0 3.14159265359 -> xyz=0.0 0.0 0.13 rpy=0 0 3.14159265359

Commit message: while testign

File: yumi_description/urdf/yumi.urdf (robot description, URDF)
Before this commit: robot yumi, 25 links, 24 joints
Joints:
- joint gripper_l_center_joint: origin xyz=0.0 0.0 0.13 rpy=0 0 3.14159265359 -> xyz=0.0 0.0 0.122 rpy=0 0 3.14159265359
- joint gripper_r_center_joint: origin xyz=0.0 0.0 0.13 rpy=0 0 3.14159265359 -> xyz=0.0 0.0 0.122 rpy=0 0 3.14159265359
- joint yumi_joint_1_l: limit lower=-2.94087978961 upper=2.94087978961 effort=300 velocity=3.14159265359 -> lower=-2.9 upper=2.9 effort=300 velocity=3.14159265359
- joint yumi_joint_1_r: limit lower=-2.94087978961 upper=2.94087978961 effort=300 velocity=3.14159265359 -> lower=-2.9 upper=2.9 effort=300 velocity=3.14159265359
- joint yumi_joint_2_l: limit lower=-2.50454747661 upper=0.759218224618 effort=300 velocity=3.14159265359 -> lower=-2.3 upper=0.70 effort=300 velocity=3.14159265359
- joint yumi_joint_2_r: limit lower=-2.50454747661 upper=0.759218224618 effort=300 velocity=3.14159265359 -> lower=-2.4 upper=0.7 effort=300 velocity=3.14159265359
- joint yumi_joint_3_l: limit lower=-2.15548162621 upper=1.3962634016 effort=300 velocity=3.14159265359 -> lower=-2.1 upper=1.3 effort=300 velocity=3.14159265359
- joint yumi_joint_3_r: limit lower=-2.15548162621 upper=1.3962634016 effort=300 velocity=3.14159265359 -> lower=-2.1 upper=1.3 effort=300 velocity=3.14159265359
- joint yumi_joint_4_l: limit lower=-5.06145483078 upper=5.06145483078 effort=300 velocity=6.98131700798 -> lower=-5.0 upper=5.0 effort=300 velocity=6.98131700798
- joint yumi_joint_4_r: limit lower=-5.06145483078 upper=5.06145483078 effort=300 velocity=6.98131700798 -> lower=-5.0 upper=5.0 effort=300 velocity=6.98131700798
- joint yumi_joint_5_l: limit lower=-1.53588974176 upper=2.40855436775 effort=300 velocity=6.98131700798 -> lower=-1.5 upper=2.4 effort=300 velocity=6.98131700798
- joint yumi_joint_5_r: limit lower=-1.53588974176 upper=2.40855436775 effort=300 velocity=6.98131700798 -> lower=-1.5 upper=2.4 effort=300 velocity=6.98131700798
- joint yumi_joint_6_l: limit lower=-3.99680398707 upper=3.99680398707 effort=300 velocity=6.98131700798 -> lower=-3.9 upper=3.9 effort=300 velocity=6.98131700798
- joint yumi_joint_6_r: limit lower=-3.99680398707 upper=3.99680398707 effort=300 velocity=6.98131700798 -> lower=-3.9 upper=3.9 effort=300 velocity=6.98131700798
- joint yumi_joint_7_l: limit lower=-2.94087978961 upper=2.94087978961 effort=300 velocity=3.14159265359 -> lower=-2.89 upper=2.89 effort=300 velocity=3.14159265359
- joint yumi_joint_7_r: limit lower=-2.94087978961 upper=2.94087978961 effort=300 velocity=3.14159265359 -> lower=-2.9 upper=2.9 effort=300 velocity=3.14159265359

Commit message: tuning

File: yumi_description/urdf/yumi.urdf (robot description, URDF)
Before this commit: robot yumi, 25 links, 24 joints
Joints:
- joint yumi_joint_2_l: limit lower=-2.3 upper=0.70 effort=300 velocity=3.14159265359 -> lower=-2.4 upper=0.7 effort=300 velocity=3.14159265359
- joint yumi_joint_7_l: limit lower=-2.89 upper=2.89 effort=300 velocity=3.14159265359 -> lower=-2.9 upper=2.9 effort=300 velocity=3.14159265359

Commit message: object handling

File: yumi_description/urdf/yumi.urdf (robot description, URDF)
Before this commit: robot yumi, 25 links, 24 joints
Joints:
- joint gripper_l_center_joint: origin xyz=0.0 0.0 0.122 rpy=0 0 3.14159265359 -> xyz=0.0 0.0 0.129 rpy=0 0 3.14159265359
- joint gripper_r_center_joint: origin xyz=0.0 0.0 0.122 rpy=0 0 3.14159265359 -> xyz=0.0 0.0 0.129 rpy=0 0 3.14159265359

Commit message: new masses

File: yumi_description/urdf/yumi.urdf (robot description, URDF)
Before this commit: robot yumi, 25 links, 24 joints
Links:
- link yumi_link_1_l: mass 2 -> 0.9629
- link yumi_link_1_r: mass 2 -> 0.9629
- link yumi_link_2_l: mass 2 -> 1.4106
- link yumi_link_2_r: mass 2 -> 1.4106
- link yumi_link_3_l: mass 2 -> 0.7108
- link yumi_link_3_r: mass 2 -> 0.7187
- link yumi_link_4_l: mass 2 -> 1.1808
- link yumi_link_4_r: mass 2 -> 1.1808
- link yumi_link_5_l: mass 2 -> 0.34345
- link yumi_link_5_r: mass 2 -> 0.34346
- link yumi_link_6_l: mass 2 -> 0.46580
- link yumi_link_6_r: mass 2 -> 0.47035
- link yumi_link_7_l: mass 2 -> 0.03094
- link yumi_link_7_r: mass 2 -> 0.04168

Commit message: tuning URDF weights

File: yumi_description/urdf/yumi.urdf (robot description, URDF)
Before this commit: robot yumi, 25 links, 24 joints
Links:
- link yumi_link_1_r: mass 0.9629 -> 1.2
- link yumi_link_2_r: mass 1.4106 -> 1.6
- link yumi_link_3_r: mass 0.7187 -> 0.9
- link yumi_link_4_r: mass 1.1808 -> 1.3
- link yumi_link_5_r: mass 0.34346 -> 0.5
- link yumi_link_6_r: mass 0.47035 -> 0.6
- link yumi_link_7_r: mass 0.04168 -> 0.24168

Commit message: tuning

File: yumi_description/urdf/yumi.urdf (robot description, URDF)
Before this commit: robot yumi, 25 links, 24 joints
Joints:
- joint gripper_l_center_joint: origin xyz=0.0 0.0 0.129 rpy=0 0 3.14159265359 -> xyz=0.0 0.0 0.131 rpy=0 0 3.14159265359
- joint gripper_r_center_joint: origin xyz=0.0 0.0 0.129 rpy=0 0 3.14159265359 -> xyz=0.0 0.0 0.131 rpy=0 0 3.14159265359

Commit message: new he

File: yumi_description/urdf/yumi.urdf (robot description, URDF)
Before this commit: robot yumi, 25 links, 24 joints
Joints:
- joint zivid_optical_joint: origin xyz=0.18817 0.06293 0.68891 rpy=-2.8595 -0.14513 -1.6163251 -> xyz=0.18957 0.063905 0.6879233 rpy=-2.7580472 -0.0675976 -2.2319674

Commit message: new he

File: yumi_description/urdf/yumi.urdf (robot description, URDF)
Before this commit: robot yumi, 25 links, 24 joints
Joints:
- joint zivid_optical_joint: origin xyz=0.18957 0.063905 0.6879233 rpy=-2.7580472 -0.0675976 -2.2319674 -> xyz=-0.6925705 0.7057567 -0.1491767 rpy=-2.8649353 -0.1455238 -1.6099504

Commit message: tuning

File: yumi_description/urdf/yumi.urdf (robot description, URDF)
Before this commit: robot yumi, 25 links, 24 joints
Joints:
- joint zivid_optical_joint: origin xyz=-0.6925705 0.7057567 -0.1491767 rpy=-2.8649353 -0.1455238 -1.6099504 -> xyz=0.18957 0.0639047 0.6879233 rpy=-2.8649353 -0.1455238 -1.6099504

Commit message: rml branch
- Applies the rml-interpolation to create additional waypoints in the segments between the Moveit 2 waypoints
- Warning, Do not work properly

File: yumi_description/urdf/yumi.urdf (robot description, URDF)
Before this commit: robot yumi, 25 links, 24 joints
Joints:
- joint yumi_joint_1_l: limit lower=-2.9 upper=2.9 effort=300 velocity=3.14159265359 -> lower=-2.7 upper=2.7 effort=300 velocity=3.14159265359
- joint yumi_joint_1_r: limit lower=-2.9 upper=2.9 effort=300 velocity=3.14159265359 -> lower=-2.7 upper=2.7 effort=300 velocity=3.14159265359
- joint yumi_joint_2_l: limit lower=-2.4 upper=0.7 effort=300 velocity=3.14159265359 -> lower=-2.4 upper=0.6 effort=300 velocity=3.14159265359
- joint yumi_joint_2_r: limit lower=-2.4 upper=0.7 effort=300 velocity=3.14159265359 -> lower=-2.4 upper=0.6 effort=300 velocity=3.14159265359
- joint yumi_joint_3_l: limit lower=-2.1 upper=1.3 effort=300 velocity=3.14159265359 -> lower=-1.9 upper=1.1 effort=300 velocity=3.14159265359
- joint yumi_joint_3_r: limit lower=-2.1 upper=1.3 effort=300 velocity=3.14159265359 -> lower=-1.9 upper=1.1 effort=300 velocity=3.14159265359
- joint yumi_joint_4_l: limit lower=-5.0 upper=5.0 effort=300 velocity=6.98131700798 -> lower=-4.8 upper=4.8 effort=300 velocity=6.98131700798
- joint yumi_joint_4_r: limit lower=-5.0 upper=5.0 effort=300 velocity=6.98131700798 -> lower=-4.8 upper=4.8 effort=300 velocity=6.98131700798
- joint yumi_joint_5_l: limit lower=-1.5 upper=2.4 effort=300 velocity=6.98131700798 -> lower=-1.4 upper=2.3 effort=300 velocity=6.98131700798
- joint yumi_joint_5_r: limit lower=-1.5 upper=2.4 effort=300 velocity=6.98131700798 -> lower=-1.4 upper=2.3 effort=300 velocity=6.98131700798
- joint yumi_joint_6_l: limit lower=-3.9 upper=3.9 effort=300 velocity=6.98131700798 -> lower=-3.7 upper=3.7 effort=300 velocity=6.98131700798
- joint yumi_joint_6_r: limit lower=-3.9 upper=3.9 effort=300 velocity=6.98131700798 -> lower=-3.7 upper=3.7 effort=300 velocity=6.98131700798
- joint yumi_joint_7_l: limit lower=-2.9 upper=2.9 effort=300 velocity=3.14159265359 -> lower=-2.7 upper=2.7 effort=300 velocity=3.14159265359
- joint yumi_joint_7_r: limit lower=-2.9 upper=2.9 effort=300 velocity=3.14159265359 -> lower=-2.7 upper=2.7 effort=300 velocity=3.14159265359

Commit message: accelerations

File: yumi_description/urdf/yumi.urdf (robot description, URDF)
Before this commit: robot yumi, 25 links, 24 joints
Joints:
- joint yumi_joint_1_l: limit lower=-2.7 upper=2.7 effort=300 velocity=3.14159265359 -> lower=-2.9 upper=2.9 effort=300 velocity=3.14159265359
- joint yumi_joint_1_r: limit lower=-2.7 upper=2.7 effort=300 velocity=3.14159265359 -> lower=-2.9 upper=2.9 effort=300 velocity=3.14159265359
- joint yumi_joint_2_l: limit lower=-2.4 upper=0.6 effort=300 velocity=3.14159265359 -> lower=-2.4 upper=0.7 effort=300 velocity=3.14159265359
- joint yumi_joint_2_r: limit lower=-2.4 upper=0.6 effort=300 velocity=3.14159265359 -> lower=-2.4 upper=0.7 effort=300 velocity=3.14159265359
- joint yumi_joint_3_l: limit lower=-1.9 upper=1.1 effort=300 velocity=3.14159265359 -> lower=-2.1 upper=1.3 effort=300 velocity=3.14159265359
- joint yumi_joint_3_r: limit lower=-1.9 upper=1.1 effort=300 velocity=3.14159265359 -> lower=-2.1 upper=1.3 effort=300 velocity=3.14159265359
- joint yumi_joint_4_l: limit lower=-4.8 upper=4.8 effort=300 velocity=6.98131700798 -> lower=-5.0 upper=5.0 effort=300 velocity=6.98131700798
- joint yumi_joint_4_r: limit lower=-4.8 upper=4.8 effort=300 velocity=6.98131700798 -> lower=-5.0 upper=5.0 effort=300 velocity=6.98131700798
- joint yumi_joint_5_l: limit lower=-1.4 upper=2.3 effort=300 velocity=6.98131700798 -> lower=-1.5 upper=2.4 effort=300 velocity=6.98131700798
- joint yumi_joint_5_r: limit lower=-1.4 upper=2.3 effort=300 velocity=6.98131700798 -> lower=-1.5 upper=2.4 effort=300 velocity=6.98131700798
- joint yumi_joint_6_l: limit lower=-3.7 upper=3.7 effort=300 velocity=6.98131700798 -> lower=-3.9 upper=3.9 effort=300 velocity=6.98131700798
- joint yumi_joint_6_r: limit lower=-3.7 upper=3.7 effort=300 velocity=6.98131700798 -> lower=-3.9 upper=3.9 effort=300 velocity=6.98131700798
- joint yumi_joint_7_l: limit lower=-2.7 upper=2.7 effort=300 velocity=3.14159265359 -> lower=-2.9 upper=2.9 effort=300 velocity=3.14159265359
- joint yumi_joint_7_r: limit lower=-2.7 upper=2.7 effort=300 velocity=3.14159265359 -> lower=-2.9 upper=2.9 effort=300 velocity=3.14159265359
